File: pcb/controlserie.sch (KiCad schematic (older format))
At the start: 55 parts

Commit message: acomodando componentes
Parts:
- removed JP?: JUMPER, symbol JUMPER
- removed R?: 2k2, Discret:R3, symbol R
- added F1: FUSE, Fuse_Holders_and_Fuses:Fuseholder5x20_horiz_SemiClosed_Casing10x25mm, symbol FUSE
- added T1: TRANSFO, locales:TFCOBSIL2209VCA200mA, symbol TRANSFO
- C1: renamed from C?; footprint Capacitors_ThroughHole:Capacitor5x11RM2.5 -> locales:C1V5
- C2, C3, C7, C8: renamed from C?; footprint Capacitors_ThroughHole:Capacitor3MMDiscRM2.5 -> locales:C1
- C4: renamed from C?; footprint (none) -> locales:C1V5
- C5: renamed from C?; footprint (none) -> locales:C1
- C6: renamed from C?; footprint Capacitors_ThroughHole:Capacitor10x16RM5 -> locales:C1V8
- D1, D6, D7, D8: renamed from D?; footprint (none) -> Diodes_ThroughHole:Diode_DO-41_SOD81_Horizontal_RM10
- D2: renamed from D?; footprint Discret:PUSH_BUTT_SHAPE1 -> locales:Bridge-rond
- D3, D4, D5: renamed from D?; footprint (none) -> LEDs:LED-5MM
- IC1: renamed from IC?; footprint Sockets_DIP:DIP-6__300_ELL -> Housings_DIP:DIP-4_W7.62mm_LongPads
- JP2: renamed from JP?; footprint (none) -> Connect:PINHEAD1-2
- K1, K2, K3: renamed from K?; footprint (none) -> Relays_ThroughHole:Relay_SANYOU_SRD_Series_Form_C
- P2: renamed from P?; value CONN_01X10 -> CON1; footprint (none) -> locales:PHOENIX_MSTBA2,54-G_10
- P3: renamed from P?; value CONN_01X03 -> CON2; footprint (none) -> locales:PHOENIX_MSTBA2,54-G_3
- P4: renamed from P?; footprint (none) -> locales:PHOENIX_MSTBA2,54-G_2
- P5: renamed from P?; value CONN_01X02 -> CON6; footprint (none) -> locales:PHOENIX_MSTBA2,54-G_2
- P6: renamed from P?; value CONN_01X03 -> DISPLAY; footprint (none) -> Connect:PINHEAD1-3
- P7: renamed from P?; value CONN_01X03 -> CON3; footprint (none) -> locales:PHOENIX_MSTBA2,54-G_3
- P8: renamed from P?; value CONN_01X03 -> CON4; footprint (none) -> locales:PHOENIX_MSTBA2,54-G_3
- P9: renamed from P?; value CONN_01X03 -> CON5; footprint (none) -> locales:PHOENIX_MSTBA2,54-G_3
- Q1, Q2, Q3: renamed from Q?; footprint SOT-23 -> TO_SOT_Packages_THT:TO-92_Molded_Narrow_Oval
- R10, R11, R13, R14, R15, R16, R17, R18, R3, R4, R5, R6, R7, R9: renamed from R?; footprint (none) -> Discret:R3
- SW1: renamed from SW?; footprint (none) -> Buttons_Switches_ThroughHole:SW_PUSH-12mm
- U1: renamed from U?; footprint Sockets_DIP:DIP-20__300_ELL -> Housings_DIP:DIP-20_W7.62mm_LongPads
- U2: renamed from U?; footprint Discret:TO92-123 -> TO_SOT_Packages_THT:TO-220_Neutral123_Horizontal
- gave numbers to parts that had none: 4
Connections:
- net labels removed: JP3
- wire segments 122 -> 125
- no-connect marks 2 -> 8
Other:
- moved on the sheet: C5, P4, P5, P6, R12
